Commit message: fixed urdf and meshses

File: rrr_description/urdf/rrr_bot.urdf (robot description, URDF)
Before this commit: robot tehreem, 4 links, 3 joints
Links:
- added link world
- link base_link: geometry collision mesh filename=package://rrr_description/meshes/base_link.STL scale=0.001 0.001 0.001; visual mesh filename=package://rrr_description/meshes/base_link.STL scale=0.001 0.001 0.001
- link link1: geometry collision mesh filename=package://rrr_description/meshes/link1.STL scale=0.001 0.001 0.001; visual mesh filename=package://rrr_description/meshes/link1.STL scale=0.001 0.001 0.001
- link link2: geometry collision mesh filename=package://rrr_description/meshes/link2.STL scale=0.001 0.001 0.001; visual mesh filename=package://rrr_description/meshes/link2.STL scale=0.001 0.001 0.001
- link link3: geometry collision mesh filename=package://rrr_description/meshes/link3.STL scale=0.001 0.001 0.001; visual mesh filename=package://rrr_description/meshes/link3.STL scale=0.001 0.001 0.001
Joints:
- added joint joint_world: type fixed, parent world, child base_link, origin xyz=0 0 0 rpy=0 0 0
